File: NU31-HackerSynth.kicad_sch (KiCad schematic)
At the start: 136 parts, among them J2 AudioJack3, J3 Barrel_Jack, J4 AudioJack2_SwitchT, J5 AudioJack2_SwitchT, J6 AudioJack2_SwitchT, J7 Eurorack Power, Q1 NPN, Q2 NPN, Q3 NPN, Q4 NPN, SW1 SW_DPDT, SW2 SW_SPDT, SW3 SW_Rotary_1x8_MP, U1 LM358, U2 LM358, U3 LM358, U4 CD4017, U5 LM358, U6 LM358, U7 LM358

Commit message: Updated and separated OSC type switch and tone control into separate blocks
Parts:
- added JP8, JP9: Jumper_2_Bridged, Connector_PinHeader_2.54mm:PinHeader_1x02_P2.54mm_Vertical, symbol Jumper:Jumper_2_Bridged
- C5: value ? -> 10n
- R34, R35: value 10k -> 1k
Connections:
- new net MIX_IN: JP8.2 (B), JP9.2 (B), RV1.1
- new net OSC1_OUT: JP8.1 (A), R34.2
- new net OSC2_OUT: JP9.1 (A), R35.2
Other:
- note added: "OSC Switch"
- moved on the sheet: C3, C4, C5, JP1, JP2, JP3, JP4, JP5, JP6, JP7, Q2, Q4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

Commit message: Added negative voltage protection for sequencer clock input, added footprints for faders and rotaryswitch
Parts:
- added D20: 1N4148, Diode_THT:D_A-405_P7.62mm_Horizontal, symbol Device:D
- added R59: 1k, Resistor_THT:R_Axial_DIN0207_L6.3mm_D2.5mm_P10.16mm_Horizontal, symbol Device:R
- J7: now not fitted
- Q1, Q2, Q3, Q4: value NPN -> BC547; symbol Simulation_SPICE:NPN -> Transistor_BJT:BC547
- RV13, RV14, RV4, RV5, RV6, RV7, RV8, RV9: footprint Potentiometer_THT:Potentiometer_Bourns_PTA2043_Single_Slide -> SpaceCow:40mm Fader Potentiometer (double)
- SW3: footprint (none) -> SpaceCow:8-way Rotary Switch
Connections:
- net GND: now also SW3.MP, D20.2 (A)
- net at U4.14 (CLK): now also D20.1 (K), R59.1; no longer SW2.2 (B)
- new net: R59.2, SW2.2 (B)
Other:
- moved on the sheet: D10, D11, D12, D13, D14, D15, D16, D17, D18, D3, D4, D5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
